Commit message: change joint names to our standard

File: robotis_op_description/urdf/arm/robotis_op_arm.urdf.xacro (robot description, xacro)
@@ -135,5 +135,5 @@
     <limit effort="2.8" velocity="5.6548668" lower="-2.6179939" upper="2.6179939" />
   </joint>
-  <joint name="j_shoulder_l" type="revolute">
+  <joint name="LShoulderPitch" type="revolute">
     <parent link="MP_BACK_L"/>
     <child link="MP_SHOULDER_L"/>
@@ -142,5 +142,5 @@
     <limit effort="2.8" velocity="5.6548668" lower="-2.6179939" upper="2.6179939" />
   </joint>
-  <joint name="j_high_arm_l" type="revolute">
+  <joint name="LShoulderRoll" type="revolute">
     <parent link="MP_SHOULDER_L"/>
     <child link="MP_ARM_HIGH_L"/>
@@ -149,5 +149,5 @@
     <limit effort="2.8" velocity="5.648668" lower="-2.6179939" upper="2.6179939" />
   </joint>
-  <joint name="j_low_arm_l" type="revolute">
+  <joint name="LElbow" type="revolute">
     <parent link="MP_ARM_HIGH_L"/>
     <child link="MP_ARM_LOW_L"/>
@@ -156,5 +156,5 @@
     <limit effort="2.8" velocity="5.6548668" lower="-2.6179939" upper="2.6179939" />
   </joint>
-  <joint name="j_wrist_l" type="revolute">
+  <joint name="j_wrist_l" type="fixed">
     <parent link="MP_ARM_LOW_L"/>
     <child link="MP_ARM_GRIPPER_FIX_L"/>
@@ -168,5 +168,5 @@
     <origin xyz="0.064 -0.01 0" rpy="0 0 0" />
   </joint>
-  <joint name="j_gripper_l" type="revolute">
+  <joint name="j_gripper_l" type="fixed">
     <parent link="MP_ARM_GRIPPER_FIX_L"/>
     <child link="MP_ARM_GRIPPER_MOV_L"/>
@@ -181,5 +181,5 @@
     <limit effort="2.8" velocity="5.6548668" lower="-2.6179939" upper="2.6179939" />
   </joint>
-  <joint name="j_shoulder_r" type="revolute">
+  <joint name="RShoulderPitch" type="revolute">
     <parent link="MP_BACK_R"/>
     <child link="MP_SHOULDER_R"/>
@@ -188,5 +188,5 @@
     <limit effort="2.8" velocity="5.6548668" lower="-2.6179939" upper="2.6179939" />
   </joint>
-  <joint name="j_high_arm_r" type="revolute">
+  <joint name="RShoulderRoll" type="revolute">
     <parent link="MP_SHOULDER_R"/>
     <child link="MP_ARM_HIGH_R"/>
@@ -195,5 +195,5 @@
     <limit effort="2.8" velocity="5.648668" lower="-2.6179939" upper="2.6179939" />
   </joint>
-  <joint name="j_low_arm_r" type="revolute">
+  <joint name="RElbow" type="revolute">
     <parent link="MP_ARM_HIGH_R"/>
     <child link="MP_ARM_LOW_R"/>
@@ -202,5 +202,5 @@
     <limit effort="2.8" velocity="5.6548668" lower="-2.6179939" upper="2.6179939" />
   </joint>
-  <joint name="j_wrist_r" type="revolute">
+  <joint name="j_wrist_r" type="fixed">
     <parent link="MP_ARM_LOW_R"/>
     <child link="MP_ARM_GRIPPER_FIX_R"/>
@@ -214,5 +214,5 @@
     <origin xyz="0.064 -0.01 0" rpy="0 0 0" />
   </joint>
-  <joint name="j_gripper_r" type="revolute">
+  <joint name="j_gripper_r" type="fixed">
     <parent link="MP_ARM_GRIPPER_FIX_R"/>
     <child link="MP_ARM_GRIPPER_MOV_R"/>
@@ -221,14 +221,10 @@
     <limit effort="2.8" velocity="5.6548668" lower="-2.6179939" upper="2.6179939" />
   </joint>
-  <joint_transmission_macro joint_name="j_shoulder_l"/>
-  <joint_transmission_macro joint_name="j_high_arm_l"/>
-  <joint_transmission_macro joint_name="j_low_arm_l"/>
-  <joint_transmission_macro joint_name="j_wrist_l"/>
-  <joint_transmission_macro joint_name="j_gripper_l"/>
-  <joint_transmission_macro joint_name="j_shoulder_r"/>
-  <joint_transmission_macro joint_name="j_high_arm_r"/>
-  <joint_transmission_macro joint_name="j_low_arm_r"/>
-  <joint_transmission_macro joint_name="j_wrist_r"/>
-  <joint_transmission_macro joint_name="j_gripper_r"/>
+  <joint_transmission_macro joint_name="LShoulderRoll"/>
+  <joint_transmission_macro joint_name="LShoulderPitch"/>
+  <joint_transmission_macro joint_name="LElbow"/>
+  <joint_transmission_macro joint_name="RShoulderRoll"/>
+  <joint_transmission_macro joint_name="RShoulderPitch"/>
+  <joint_transmission_macro joint_name="RElbow"/>
   </macro>
 </robot>
