Commit message: joint limits

File: darwin_description/urdf/arm/darwin_arm.urdf.xacro (robot description, xacro)
@@ -140,5 +140,5 @@
     <origin xyz="0 0 0" rpy="0 0 -1.5707963" />
     <axis xyz="0 0 1" />
-    <limit effort="2.8" velocity="5.6548668" lower="-2.6179939" upper="2.6179939" />
+    <limit effort="2.8" velocity="5.6548668" lower="-3.14" upper="2.85" />
   </joint>
   <joint name="LShoulderRoll" type="revolute">
@@ -147,5 +147,5 @@
     <origin xyz="-0.016 0 0.02165" rpy="1.5707963 0.78539815 0" />
     <axis xyz="0 0 1" />
-    <limit effort="2.8" velocity="5.648668" lower="-2.6179939" upper="2.6179939" />
+    <limit effort="2.8" velocity="5.648668" lower="-2.25" upper="0.77" />
   </joint>
   <joint name="LElbow" type="revolute">
@@ -154,5 +154,5 @@
     <origin xyz="-0.06 0 -0.016" rpy="-1.5707963 1.5707963 0" />
     <axis xyz="0 0 1" />
-    <limit effort="2.8" velocity="5.6548668" lower="-2.6179939" upper="2.6179939" />
+    <limit effort="2.8" velocity="5.6548668" lower="-1.18" upper="1.63" />
   </joint>
   <joint name="j_wrist_l" type="fixed">
@@ -186,5 +186,5 @@
     <origin xyz="0 0 0" rpy="0 0 1.5707963" />
     <axis xyz="0 0 1" />
-    <limit effort="2.8" velocity="5.6548668" lower="-2.6179939" upper="2.6179939" />
+    <limit effort="2.8" velocity="5.6548668" lower="-3.14" upper="3.14" />
   </joint>
   <joint name="RShoulderRoll" type="revolute">
@@ -193,5 +193,5 @@
     <origin xyz="-0.016 0 0.02165" rpy="-1.5707963 0.78539815 0" />
     <axis xyz="0 0 1" />
-    <limit effort="2.8" velocity="5.648668" lower="-2.6179939" upper="2.6179939" />
+    <limit effort="2.8" velocity="5.648668" lower="-0.68" upper="2.3" />
   </joint>
   <joint name="RElbow" type="revolute">
@@ -200,5 +200,5 @@
     <origin xyz="-0.06 0 -0.016" rpy="1.5707963 1.5707963 0" />
     <axis xyz="0 0 1" />
-    <limit effort="2.8" velocity="5.6548668" lower="-2.6179939" upper="2.6179939" />
+    <limit effort="2.8" velocity="5.6548668" lower="-1.65" upper="1.16" />
   </joint>
   <joint name="j_wrist_r" type="fixed">
