Commit message: fixes

File: darwin_description/urdf/robot.urdf (robot description, URDF)
Before this commit: robot darwin, 31 links, 30 joints
Links:
- added link MP_ANKLE2_L, mass 0.0794462; collision box size=0.008 0.066 0.104; visual mesh filename=package://darwin_description/meshes/ankle2_l.STL scale=1 1 1
- added link MP_ANKLE2_R, mass 0.0794462; collision box size=0.008 0.066 0.104; visual mesh filename=package://darwin_description/meshes/ankle2_r.STL scale=1 1 1
- link l_sole: mass 0.0794462 -> None; geometry 
- link r_sole: mass 0.0794462 -> None; geometry 
Joints:
- added joint l_sole_joint: type fixed, parent MP_ANKLE2_L, child l_sole, origin xyz=-0.033 -0.01 0 rpy=3.14 -1.57 0
- added joint r_sole_joint: type fixed, parent MP_ANKLE2_R, child r_sole, origin xyz=0.033 -0.01 0 rpy=0 -1.57 0
- joint HeadPan: limit lower=-2.6179939 upper=2.6179939 effort=2.8 velocity=5.6548668 -> lower=-1.81 upper=1.81 effort=2.8 velocity=5.6548668
- joint HeadTilt: limit lower=-2.6179939 upper=2.6179939 effort=2.8 velocity=5.6548668 -> lower=-0.36 upper=0.94 effort=2.8 velocity=5.6548668
- joint LAnklePitch: limit lower=-2.6179939 upper=2.6179939 effort=2.8 velocity=5.6548668 -> lower=-1.39 upper=1.22 effort=2.8 velocity=5.6548668
- joint LAnkleRoll: child l_sole -> MP_ANKLE2_L; limit lower=-2.6179939 upper=2.6179939 effort=2.8 velocity=5.6548668 -> lower=-1.02 upper=0.6 effort=2.8 velocity=5.6548668
- joint LElbow: limit lower=-2.6179939 upper=2.6179939 effort=2.8 velocity=5.6548668 -> lower=-1.18 upper=1.63 effort=2.8 velocity=5.6548668
- joint LHipPitch: limit lower=-2.6179939 upper=2.6179939 effort=2.8 velocity=5.6548668 -> lower=-0.5 upper=1.68 effort=2.8 velocity=5.6548668
- joint LHipRoll: limit lower=-2.6179939 upper=2.6179939 effort=2.8 velocity=5.6548668 -> lower=-1 upper=0.93 effort=2.8 velocity=5.6548668
- joint LHipYaw: limit lower=-2.6179939 upper=2.6179939 effort=2.8 velocity=5.6548668 -> lower=-0.69 upper=2.5 effort=2.8 velocity=5.6548668
- joint LKnee: limit lower=-2.6179939 upper=2.6179939 effort=2.8 velocity=5.6548668 -> lower=-2.25 upper=0.0 effort=2.8 velocity=5.6548668
- joint LShoulderPitch: limit lower=-2.6179939 upper=2.6179939 effort=2.8 velocity=5.6548668 -> lower=-3.14 upper=2.85 effort=2.8 velocity=5.6548668
- joint LShoulderRoll: limit lower=-2.6179939 upper=2.6179939 effort=2.8 velocity=5.648668 -> lower=-2.25 upper=0.77 effort=2.8 velocity=5.648668
- joint RAnklePitch: limit lower=-2.6179939 upper=2.6179939 effort=2.8 velocity=5.6548668 -> lower=-1.24 upper=1.38 effort=2.8 velocity=5.6548668
- joint RAnkleRoll: child r_sole -> MP_ANKLE2_R; limit lower=-2.6179939 upper=2.6179939 effort=2.8 velocity=5.6548668 -> lower=-0.68 upper=1.04 effort=2.8 velocity=5.6548668
- joint RElbow: limit lower=-2.6179939 upper=2.6179939 effort=2.8 velocity=5.6548668 -> lower=-1.65 upper=1.16 effort=2.8 velocity=5.6548668
- joint RHipPitch: limit lower=-2.6179939 upper=2.6179939 effort=2.8 velocity=5.6548668 -> lower=-1.77 upper=0.45 effort=2.8 velocity=5.6548668
- joint RHipRoll: limit lower=-2.6179939 upper=2.6179939 effort=2.8 velocity=5.6548668 -> lower=-1.01 upper=1.01 effort=2.8 velocity=5.6548668
- joint RHipYaw: limit lower=-2.6179939 upper=2.6179939 effort=2.8 velocity=5.6548668 -> lower=-2.42 upper=0.66 effort=2.8 velocity=5.6548668
- joint RKnee: limit lower=-2.6179939 upper=2.6179939 effort=2.8 velocity=5.6548668 -> lower=0 upper=2.25 effort=2.8 velocity=5.6548668
- joint RShoulderPitch: limit lower=-2.6179939 upper=2.6179939 effort=2.8 velocity=5.6548668 -> lower=-3.14 upper=3.14 effort=2.8 velocity=5.6548668
- joint RShoulderRoll: limit lower=-2.6179939 upper=2.6179939 effort=2.8 velocity=5.648668 -> lower=-0.68 upper=2.3 effort=2.8 velocity=5.648668
- joint base_link_to_body: origin xyz=0 0 0.35 rpy=0 0 0 -> xyz=0.005 0 0.09355 rpy=0 0 0

File: darwin_description/urdf/torso/darwin_torso.urdf.xacro (robot description, xacro)
@@ -16,5 +16,5 @@
     <parent link="base_link"/>
     <child link="MP_BODY"/>
-    <origin xyz="0 0 0.35" rpy="0 0 0"/>
+    <origin xyz="0.005 0 0.09355" rpy="0 0 0"/>
   </joint>
       <gazebo>

Commit message: fixes an urdf

File: darwin_description/urdf/robot.urdf (robot description, URDF)
Before this commit: robot darwin, 33 links, 32 joints
Links:
- added link imu_frame
Joints:
- added joint base_link_to_imu: type fixed, parent base_link, child imu_frame, origin xyz=0 0 0 rpy=0 0 0

File: darwin_description/urdf/torso/darwin_torso.urdf.xacro (robot description, xacro)
@@ -4,4 +4,5 @@
   <macro name="darwin_torso_macro">
   <link name="base_link"/>
+  <link name="imu_frame"/>
   <link name="MP_BODY">
     <inertial>
@@ -18,4 +19,9 @@
     <origin xyz="0.005 0 0.09355" rpy="0 0 0"/>
   </joint>
+  <joint name="base_link_to_imu" type="fixed">
+    <parent link="base_link"/>
+    <child link="imu_frame"/>
+    <origin xyz="0 0 0" rpy="0 0 0"/>
+  </joint>
       <gazebo>
         <plugin filename="libhector_gazebo_ros_imu.so" name="gazebo_ros_imu">

Commit message: links for walking

File: darwin_description/urdf/robot.urdf (robot description, URDF)
Before this commit: robot darwin, 34 links, 33 joints
Links:
- link base_link: mass None -> 1e-9
- link imu_frame: mass None -> 1e-9
- link l_sole: mass None -> 1e-9
- link r_sole: mass None -> 1e-9

Commit message: urdf fix

File: darwin_description/urdf/robot.urdf (robot description, URDF)
Before this commit: robot darwin, 34 links, 33 joints
Links:
- link MP_PMDCAMBOARD: mass None -> 1e-9
- link base_link: mass None -> 1e-9
- link imu_frame: mass None -> 1e-9
- link l_sole: mass None -> 1e-9
- link r_sole: mass None -> 1e-9

Commit message: fix darwin head rotation

File: darwin_description/urdf/robot.urdf (robot description, URDF)
Before this commit: robot darwin, 34 links, 33 joints
Joints:
- joint HeadTilt: origin xyz=0 0 0.02715 rpy=-1.5707963 0 1.5707963 -> xyz=0 0 0.02715 rpy=-1.5707963 0.75 1.5707963
